File: Documents/Eagle/x0x - midi daughter schematic.sch (EAGLE design)
At the start: 5 parts, among them IC3 74HC04N

Commit message: Fix last electronic issue
Updated few documents
Parts:
- removed DAC: MAX526CNG, maxim:MAX526CNG
- removed IC3: 74HC04N, 74xx-eu:74HC04N
- removed SERIAL-PARALLEL: 74HC595N, 74xx-eu:74HC595N
- added U$1: MCP4922-E/P, Microchip_By_element14_Batch_1:MCP4922-E/P
Connections:
- removed net N$10: MICRO-CONTROLER.11, SERIAL-PARALLELA.SCK
- removed net N$11: MICRO-CONTROLER.10, SERIAL-PARALLELA.SCL
- removed net N$13: DAC.CSMSB, MICRO-CONTROLER.4
- removed net N$14: DAC.CSLSB, MICRO-CONTROLER.13
- removed net N$15: DAC.WR, MICRO-CONTROLER.5
- removed net N$16: DAC.LDAC, MICRO-CONTROLER.7
- removed net N$17: DAC.A0, MICRO-CONTROLER.8
- removed net N$18: DAC.A1, MICRO-CONTROLER.9
- removed net N$5 (its old number): DAC.D4, SERIAL-PARALLELA.QE
- removed net N$6: DAC.D5, SERIAL-PARALLELA.QF
- removed net N$8: DAC.D7, SERIAL-PARALLELA.QH
- removed net N$9: MICRO-CONTROLER.12, SERIAL-PARALLELA.RCK
- net N$1: now also MICRO-CONTROLER.21, U$1.SCK; no longer DAC.D0/D8, SERIAL-PARALLELA.QA
- net N$2: now also MICRO-CONTROLER.22, U$1.SDI; no longer DAC.D1/D9, SERIAL-PARALLELA.QB
- net N$3: now also MICRO-CONTROLER.10, U$1.~CS; no longer DAC.D2/D10, SERIAL-PARALLELA.QC
- net N$4: now also MICRO-CONTROLER.VCC, OPTO-COUPLER.VCC, U$1.VDD, U$1.VREFA, U$1.VREFB; no longer DAC.D3/D11, SERIAL-PARALLELA.QD
- net N$7: now also MICRO-CONTROLER.GND, OPTO-COUPLER.GND, U$1.AVSS, U$1.~SHDN; no longer DAC.D6, SERIAL-PARALLELA.QG
Other:
- moved on the sheet: OPTO-COUPLER
