File: Documents/Eagle/x0x - midi daughter schematic.sch (EAGLE design)
At the start: 7 parts

Commit message: Add missing digital controls for x0x
Added some code, pinout draw updated and few components added on EAGLE
Parts:
- added R3: 220, rcl:R-US_0204/7
Connections:
- new net N$7: MICRO-CONTROLER.5, R3.1
Other:
- note added: "LED"
- note added: "MIDI IN 1"
- note added: "MIDI IN 2"
Changed lines of the file:
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@@
 <part name="AGND1" library="supply1" deviceset="AGND" device=""/>
 <part name="C1" library="rcl" deviceset="CPOL-EU" device="E1.8-4" value="10 µF"/>
+<part name="R3" library="rcl" deviceset="R-US_" device="0204/7" value="220"/>
 </parts>
 <sheets>
 <sheet>
 <plain>
+<text x="5.08" y="86.36" size="1.778" layer="91">LED</text>
+<text x="-30.48" y="50.8" size="1.778" layer="91">MIDI IN 1</text>
+<text x="-30.48" y="27.94" size="1.778" layer="91">MIDI IN 2</text>
 </plain>
 <instances>
@@
 <instance part="AGND1" gate="VR1" x="83.82" y="40.64"/>
 <instance part="C1" gate="G$1" x="10.16" y="144.78" rot="R180"/>
+<instance part="R3" gate="G$1" x="2.54" y="83.82"/>
 </instances>
 <busses>
@@
 <pinref part="D1" gate="G$1" pin="A"/>
 <wire x1="-5.08" y1="33.02" x2="-5.08" y2="35.56" width="0.1524" layer="91"/>
+<wire x1="-5.08" y1="33.02" x2="-20.32" y2="33.02" width="0.1524" layer="91"/>
+<junction x="-5.08" y="33.02"/>
 </segment>
 </net>
+<net name="N$7" class="0">
+<segment>
+<pinref part="MICRO-CONTROLER" gate="G$1" pin="5"/>
+<wire x1="-7.62" y1="83.82" x2="-2.54" y2="83.82" width="0.1524" layer="91"/>
+<pinref part="R3" gate="G$1" pin="1"/>
+</segment>
+</net>

Commit message: Finalise PCB
Finish PCB v 1.0
Parts:
- added +5V, ACCENT, DECAY, GROUND, LED, MIDI1, MIDI2, SAW+, SAW_IN, SAW_OUT, SLIDE_IN, SLIDE_OUT, SQUARE+, SQUARE_IN, SQUARE_OUT, UNUSED, VCF_GATE, VCO, VCO_GATE: (no value), rcl:R-US_0207/10
- added R4, R5: 10K, rcl:R-US_0207/10
- renumbered U$1 to DAC
Connections:
- new net N$10: LED.2, R3.2
- new net N$11: DAC.VOUTA, VCO.2
- new net N$12: DAC.VOUTB, UNUSED.2
- new net N$13: MICRO-CONTROLER.8, SLIDE_IN.2
- new net N$14: DECAY.2, MICRO-CONTROLER.4
- new net N$15: ACCENT.2, MICRO-CONTROLER.7
- new net N$16: MICRO-CONTROLER.9, VCO_GATE.2
- new net N$17: MICRO-CONTROLER.17, VCF_GATE.2
- new net N$18: MICRO-CONTROLER.13, R4.1, SQUARE_IN.2
- new net N$19: MICRO-CONTROLER.14,PWM, R5.1, SAW_IN.2
- new net N$20: SAW+.1
- new net N$21: SAW_IN.1
- new net N$22: SQUARE+.1
- new net N$23: MICRO-CONTROLER.15,PWM, SQUARE_OUT.2
- new net N$24: MICRO-CONTROLER.16,PWM, SAW_OUT.2
- new net N$25: SQUARE_IN.1
- new net N$26: +5V.1
- new net N$27: GROUND.1
- new net N$28: SAW_OUT.1
- new net N$29: SQUARE_OUT.1
- new net N$30: VCF_GATE.1
- new net N$31: VCO_GATE.1
- new net N$32: ACCENT.1
- new net N$33: DECAY.1
- new net N$34: SLIDE_OUT.1
- new net N$35: SLIDE_IN.1
- new net N$36: UNUSED.1
- new net N$37: VCO.1
- new net N$38: LED.1
- new net N$39: MIDI2.1
- new net N$40: MIDI1.1
- new net N$41: DAC.~LDAC
- new net N$42: DAC.NC_2
- new net N$43: DAC.NC_3
- new net N$44: DAC.NC
- new net N$45: MICRO-CONTROLER.11
- new net N$46: MICRO-CONTROLER.6,LED
- new net N$47: MICRO-CONTROLER.3,TX,INT3
- new net N$48: MICRO-CONTROLER.1,PWM,INT1
- new net N$49: MICRO-CONTROLER.0,PWM,INT0
- new net N$50: MICRO-CONTROLER.27,PWM
- new net N$8: MIDI1.2, R1.1
- new net N$9: MICRO-CONTROLER.12, SLIDE_OUT.2
- net +5V: now also +5V.2, SAW+.2, SQUARE+.2
- net AGND: now also GROUND.2, R4.2, R5.2
- net N$4: now also MIDI2.2
Other:
- moved on the sheet: R2, R3
