File: Documents/Eagle/x0x - midi daughter schematic.brd (EAGLE design)
At the start: 98.8 x 69.9 mm, 29 parts

Commit message: Fix DAC shutdown/latch wiring, revise firmware, document changes
Schematic (.sch) — netlist corrections (verified by re-parse, ERC/DRC
still required in Eagle):
- MCP4922 ~SHDN (pin 9) moved from AGND to +5V. It was tied to ground,
  which holds both DAC outputs in permanent hardware shutdown.
- ~LDAC (pin 8) now wired to MCU pin 11; both were floating stubs, so
  the DAC latch line was never connected.
- VOUTB connector pad renamed UNUSED -> VCF_CUTOFF (.sch + .brd) to
  document the VCF cutoff output intent.

NOTE: board copper was intentionally NOT hand-edited — moving the ~SHDN
net while leaving old traces would short +5V to GND. The .brd is left
for Eagle to reconcile (ERC -> forward-annotate -> re-route ~SHDN and
~LDAC airwires -> DRC).

Firmware (.ino):
- WriteDAC(channel, value) builds the 16-bit word per channel, enabling
  channel B (VCF); VCF cutoff driven from MIDI CC 74.
- Non-blocking LED blink (millis) removes 25 ms gate latency on Note On.
- Monophonic note stack (last-note priority) prevents Note Off of an
  inactive note from cutting the gate.
- MIDI input filtered to MIDIChannel instead of OMNI.
- Removed dead code (shadowed `type`, unused Uart, stray PIN_D2/PIN_D3).

README updated to match.

Co-Authored-By: Claude Opus 4.8 <noreply@anthropic.com>
Parts:
- renumbered UNUSED to VCF_CUTOFF
Changed lines of the file:
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@@
 <element name="LED" library="rcl" package="0207/10" value="" x="20.24" y="52.88"/>
 <element name="VCO" library="rcl" package="0207/10" value="" x="20.24" y="47.8"/>
-<element name="UNUSED" library="rcl" package="0207/10" value="" x="20.24" y="42.72"/>
+<element name="VCF_CUTOFF" library="rcl" package="0207/10" value="" x="20.24" y="42.72"/>
 <element name="SLIDE_IN" library="rcl" package="0207/10" value="" x="20.24" y="37.64"/>
 <element name="SLIDE_OUT" library="rcl" package="0207/10" value="" x="20.24" y="32.56"/>
@@
 <signal name="N$12">
 <contactref element="DAC" pad="10"/>
-<contactref element="UNUSED" pad="2"/>
+<contactref element="VCF_CUTOFF" pad="2"/>
 <wire x1="50.8" y1="43.18" x2="25.4" y2="43.18" width="0.1524" layer="16"/>
 <wire x1="54.61" y1="46.99" x2="50.8" y2="43.18" width="0.1524" layer="16"/>
@@
 </signal>
 <signal name="N$36">
-<contactref element="UNUSED" pad="1"/>
+<contactref element="VCF_CUTOFF" pad="1"/>
 </signal>
 <signal name="N$37">

Commit message: Make board netlist consistent with fixed schematic; update PCB notes
Board (.brd) — bring the netlist in line with the corrected schematic, as a
clean ECO (no shorts, two nets left as airwires for re-routing in Eagle):
- ~SHDN (DAC pad 9) moved from AGND to +5V signal.
- Removed the AGND copper that reached pad 9 (no ground pour exists), so the
  pad is fully isolated and becomes an unrouted airwire instead of a short.
- ~LDAC merged: MCU pin 11 (pad C1) added to the DAC pad-8 net; old N$45 removed.
- AVSS (pad 12) copper left intact.

Verified by re-parse: .brd netlist now matches .sch (~SHDN in +5V, AVSS in
AGND, ~LDAC = DAC.8 + MICRO.C1), and no copper touches pad 9.

README: PCB notes updated to reflect the netlist fixes and the remaining
Eagle step (route ~SHDN and ~LDAC airwires + DRC before fab).

Co-Authored-By: Claude Opus 4.8 <noreply@anthropic.com>
Connections:
- removed net N$45: MICRO-CONTROLER.C1
- net +5V: now also DAC.9
- net AGND: no longer DAC.9
- net N$41: now also MICRO-CONTROLER.C1
Routing:
- net AGND: track 116.1 -> 114.1 mm
Changed lines of the file:
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@@
 <signal name="+5V">
 <contactref element="MICRO-CONTROLER" pad="+5V"/>
+<contactref element="DAC" pad="9"/>
 <contactref element="DAC" pad="1"/>
 <contactref element="DAC" pad="11"/>
@@
 <signal name="AGND">
 <contactref element="C1" pad="-"/>
-<contactref element="DAC" pad="9"/>
 <contactref element="DAC" pad="12"/>
 <contactref element="OPTO-COUPLER" pad="5"/>
@@
 <wire x1="30.48" y1="62.23" x2="29.4" y2="62.04" width="0.1524" layer="16"/>
 <wire x1="50.8" y1="62.23" x2="50.609" y2="62.04" width="0.1524" layer="16"/>
-<wire x1="62.23" y1="46.99" x2="63.5" y2="45.72" width="0.1524" layer="1"/>
 <wire x1="62.23" y1="54.61" x2="62.23" y2="46.99" width="0.1524" layer="1"/>
-<wire x1="63.5" y1="45.72" x2="63.69" y2="45.8" width="0.1524" layer="1"/>
 <wire x1="60.96" y1="26.67" x2="62.23" y2="25.4" width="0.1524" layer="1"/>
 <wire x1="60.96" y1="62.23" x2="60.96" y2="26.67" width="0.1524" layer="1"/>
@@
 <signal name="N$41">
 <contactref element="DAC" pad="8"/>
+<contactref element="MICRO-CONTROLER" pad="C1"/>
 </signal>
 <signal name="N$42">
@@
 <contactref element="DAC" pad="7"/>
 </signal>
-<signal name="N$45">
-<contactref element="MICRO-CONTROLER" pad="C1"/>
-</signal>
 <signal name="N$46">

Commit message: Remove dangling AGND stub near DAC pad 9 on the board
Left over after isolating ~SHDN from AGND: a 7.62 mm AGND track ended in
mid-air at (62.23,46.99). AVSS stays connected via the (63.5,53.34) node,
so the stub was pure dead copper. Verified with KiCad DRC (kicad-cli pcb
import --format eagle + drc): the track_dangling violation is gone and the
only remaining unconnected items are the two intended airwires (~SHDN->+5V,
pin 11->~LDAC). No shorts, no schematic-parity errors.

Co-Authored-By: Claude Opus 4.8 <noreply@anthropic.com>
Routing:
- net AGND: track 114.1 -> 106.4 mm
Changed lines of the file:
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@@
 <wire x1="30.48" y1="62.23" x2="29.4" y2="62.04" width="0.1524" layer="16"/>
 <wire x1="50.8" y1="62.23" x2="50.609" y2="62.04" width="0.1524" layer="16"/>
-<wire x1="62.23" y1="54.61" x2="62.23" y2="46.99" width="0.1524" layer="1"/>
 <wire x1="60.96" y1="26.67" x2="62.23" y2="25.4" width="0.1524" layer="1"/>
 <wire x1="60.96" y1="62.23" x2="60.96" y2="26.67" width="0.1524" layer="1"/>
